File: mitsubishi-cn105-controller/mitsubishi-cn105-controller.kicad_pcb (KiCad board)
At the start: 2 copper layers, 26 x 48.8 mm, 29 parts, among them J1 Conn_01x04, J2 USB_OTG, J3 Screw_Terminal_01x04, J4 Conn_01x05_Pin, Q1 BSS138, Q2 BSS138, SW1 SW_Push, SW2 SW_Push, U1 ESP32-C3-WROOM-02, U2 AP2112K-3.3

Commit message: Very quick basic board layout
Parts:
- removed J1: Conn_01x04, Connector_PinHeader_2.54mm:PinHeader_1x04_P2.54mm_Vertical
- removed J3: Screw_Terminal_01x04, TerminalBlock_Phoenix:TerminalBlock_Phoenix_MPT-0,5-4-2.54_1x04_P2.54mm_Horizontal
- C6, C7, J2, R1, R2, R3, R4, R5, R6, R7: moved to B.Cu
- D2, D3: moved to F.Cu
- moved C4 65.8 mm to (107.6, 47.6), turned to 90 degrees
- moved D2 63.2 mm to (113.5, 44.2), turned to 90 degrees
- moved D3 61.2 mm to (111.9, 44.2), turned to 90 degrees
- moved C1 56.6 mm to (97.3, 46.9)
- moved C2 56.4 mm to (97.3, 44.8)
- moved R5 56.3 mm to (107.1, 55.8), turned to -90 degrees
- moved Q1 56.0 mm to (102.8, 58.6)
- moved Q2 56.0 mm to (102.7, 55.0)
- moved C5 55.3 mm to (97.3, 49.0)
- moved R8 53.5 mm to (113.5, 41.1), turned to 90 degrees
- moved J4 53.3 mm to (112.9, 48.5)
- moved R6 52.7 mm to (105.6, 54.1), turned to -90 degrees
- moved U2 52.6 mm to (103.7, 49.8), turned to 180 degrees
- moved D1 51.6 mm to (109.3, 56.4), turned to -90 degrees
- moved R9 51.5 mm to (111.9, 41.1), turned to -90 degrees
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Connections:
- U1 pad 11: Net-(J1-Pin_3) -> unconnected-(U1-IO20/RXD-Pad11)
- U1 pad 12: Net-(J1-Pin_2) -> unconnected-(U1-IO21/TXD-Pad12)
- U1 pad 17: Net-(J3-Pin_4) -> unconnected-(U1-IO1-Pad17)
- U1 pad 18: Net-(J3-Pin_3) -> unconnected-(U1-IO0-Pad18)
Routing:
- net +3V3: track 0.00 -> 45.3 mm, vias 0 -> 2
- net GPIO19: track 0.00 -> 22.2 mm, vias 0 -> 1
- net E32_TX_MIT_RX: track 0.00 -> 20.9 mm, vias 0 -> 1
- net GPIO18: track 0.00 -> 20.3 mm, vias 0 -> 1
- net E32_RX_MIT_TX: track 0.00 -> 15.4 mm, vias 0 -> 1
- net Net-(C7-Pad1): track 0.00 -> 13.2 mm, vias 0 -> 1
- net E32_TX_MIT_RX_5V: track 0.00 -> 10.9 mm
- net E32_RX_MIT_TX_5V: track 0.00 -> 9.74 mm
- net Net-(D1-A): track 0.00 -> 9.65 mm
- net GND: track 0.00 -> 7.38 mm, vias 0 -> 1
- net Net-(U1-IO9): track 0.00 -> 6.48 mm
- net EN: track 0.00 -> 5.20 mm, vias 0 -> 1
- net LED: track 0.00 -> 3.51 mm
- net Net-(U1-IO2): track 0.00 -> 1.89 mm, vias 0 -> 1
- net Net-(D3-A): track 0.00 -> 1.48 mm
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- added copper zone on B.Cu, net +3V3
- added copper zone on B.Cu, net +5V
- removed copper zone on F.Cu, net (none)
- removed copper zone on F.Cu, net +3V3
Other:
- board size 26 x 48.8 mm -> 27.9 x 48.8 mm

Commit message: Close to v1 complete.
Routing:
- net GND: track 7.38 -> 20.7 mm, vias 1 -> 11
Other:
- board size 27.9 x 48.8 mm -> 27.9 x 33.2 mm
